Commit message: Jazzy migration (2/6): port URDF/xacro sim plugins to Gazebo Harmonic
- gazebo.xacro: gazebo_ros2_control -> gz_ros2_control-system plugin;
  libgazebo_ros_p3d ground truth -> gz-sim OdometryPublisher system;
  libgazebo_ros_imu_sensor -> native gz-sim IMU topic (no plugin needed,
  bridged via ros_gz_bridge instead); added <sensor type="contact"> on
  each foot link, feeding the rewritten contact_sensor node.
- leg.xacro: ros2_control hardware plugin gazebo_ros2_control/GazeboSystem
  -> gz_ros2_control/GazeboSimSystem.
- laser.xacro / velodyne.xacro: Classic 'ray' sensor + gazebo_ros_ray_sensor /
  libgazebo_ros_velodyne_laser plugins -> native Harmonic 'gpu_lidar' sensor
  type, published over gz transport and bridged to ROS via ros_gz_bridge
  (see champ_gazebo/config/*_bridge.yaml added in the next commit).

File: robots/descriptions/go2_description/xacro/gazebo.xacro (robot description, xacro)
@@ -1,19 +1,20 @@
 <?xml version="1.0"?>
 <robot>
+    <!-- Ground truth odometry. Gazebo Classic's libgazebo_ros_p3d.so has no
+         Harmonic equivalent; gz-sim publishes ground-truth pose via its own
+         OdometryPublisher system on a gz transport topic, which is bridged
+         to ROS as nav_msgs/Odometry on "odom/ground_truth" by
+         champ_gazebo/config/*_bridge.yaml. -->
     <gazebo>
-      <plugin name="p3d_base_controller" filename="libgazebo_ros_p3d.so">
-        <ros>
-            <remapping>odom:=odom/ground_truth</remapping>
-        </ros>
-        <body_name>base_link</body_name>
-        <frame_name>world</frame_name>
-        <update_rate>10.0</update_rate>
-        <xyz_offset>0 0 0</xyz_offset>
-        <rpy_offset>0 0 0</rpy_offset>
-        <gaussian_noise>0.01</gaussian_noise>
-    </plugin>
+        <plugin filename="gz-sim-odometry-publisher-system" name="gz::sim::systems::OdometryPublisher">
+            <odom_frame>world</odom_frame>
+            <robot_base_frame>base_link</robot_base_frame>
+            <odom_topic>odom/ground_truth</odom_topic>
+            <odom_publish_frequency>10</odom_publish_frequency>
+            <dimensions>3</dimensions>
+        </plugin>
     </gazebo>
     <gazebo>
-        <plugin filename="libgazebo_ros2_control.so" name="gazebo_ros2_control">
+        <plugin filename="gz_ros2_control-system" name="gz_ros2_control::GazeboSimROS2ControlPlugin">
         <parameters>$(find go2_description)/config/ros_control/ros_control.yaml</parameters>
       </plugin>
@@ -21,6 +22,12 @@
     <gazebo reference="imu_link">
         <sensor name="imu_sensor" type="imu">
+            <!-- Gazebo Harmonic's IMU sensor publishes natively on a gz
+                 transport topic; no plugin is required (unlike Gazebo
+                 Classic's libgazebo_ros_imu_sensor.so). champ_gazebo bridges
+                 this topic to sensor_msgs/Imu on "imu/data". -->
             <always_on>true</always_on>
             <update_rate>100</update_rate>
+            <topic>imu</topic>
+            <gz_frame_id>imu_link</gz_frame_id>
             <imu>
             <angular_velocity>
@@ -65,11 +72,44 @@
             </linear_acceleration>
             </imu>
-            <plugin name="imu_plugin" filename="libgazebo_ros_imu_sensor.so">
-                <ros>
-                    <namespace>imu</namespace>
-                    <remapping>~/out:=data</remapping>
-                </ros>
-                <initial_orientation_as_reference>false</initial_orientation_as_reference>
-            </plugin>
+        </sensor>
+    </gazebo>
+    <!-- Foot contact sensors, read by champ_gazebo's contact_sensor node via
+         ros_gz_bridge (see champ_gazebo/config/contact_bridge.yaml). Gazebo
+         Classic's contact state was read out-of-band via gazebo::transport;
+         Harmonic exposes it as a first-class <sensor type="contact">. -->
+    <gazebo reference="lf_foot_link">
+        <sensor name="lf_foot_contact" type="contact">
+            <always_on>true</always_on>
+            <update_rate>50</update_rate>
+            <contact>
+                <collision>lf_foot_link_collision</collision>
+            </contact>
+        </sensor>
+    </gazebo>
+    <gazebo reference="rf_foot_link">
+        <sensor name="rf_foot_contact" type="contact">
+            <always_on>true</always_on>
+            <update_rate>50</update_rate>
+            <contact>
+                <collision>rf_foot_link_collision</collision>
+            </contact>
+        </sensor>
+    </gazebo>
+    <gazebo reference="lh_foot_link">
+        <sensor name="lh_foot_contact" type="contact">
+            <always_on>true</always_on>
+            <update_rate>50</update_rate>
+            <contact>
+                <collision>lh_foot_link_collision</collision>
+            </contact>
+        </sensor>
+    </gazebo>
+    <gazebo reference="rh_foot_link">
+        <sensor name="rh_foot_contact" type="contact">
+            <always_on>true</always_on>
+            <update_rate>50</update_rate>
+            <contact>
+                <collision>rh_foot_link_collision</collision>
+            </contact>
         </sensor>
     </gazebo>

File: robots/descriptions/go2_description/xacro/laser.xacro (robot description, xacro)
@@ -26,11 +26,18 @@
         </inertial>
     </link>
+    <!-- Gazebo Harmonic has no libgazebo_ros_ray_sensor.so plugin. The
+         gpu_lidar sensor type publishes sensor_msgs-compatible scans
+         natively over gz transport; champ_gazebo's ros_gz_bridge config
+         (config/laser_bridge.yaml) republishes the "scan" topic as a ROS 2
+         sensor_msgs/LaserScan. -->
     <gazebo reference="front_laser">
-        <sensor name="front_laser_sensor" type="ray">
+        <sensor name="front_laser_sensor" type="gpu_lidar">
             <always_on>true</always_on>
             <visualize>false</visualize>
             <pose>-0.032 0 0.171 0 0 0</pose>
             <update_rate>50</update_rate>
-            <ray>
+            <topic>scan</topic>
+            <gz_frame_id>front_laser</gz_frame_id>
+            <lidar>
             <scan>
                 <horizontal>
@@ -51,12 +58,5 @@
                 <stddev>0.01</stddev>
             </noise>
-            </ray>
-            <plugin name="gazebo_ros_front_laserscan" filename="libgazebo_ros_ray_sensor.so">
-            <ros>
-                <remapping>~/out:=scan</remapping>
-            </ros>
-            <output_type>sensor_msgs/LaserScan</output_type>
-            <frame_name>front_laser</frame_name>
-            </plugin>
+            </lidar>
         </sensor>
     </gazebo>

File: robots/descriptions/go2_description/xacro/leg.xacro (robot description, xacro)
@@ -157,5 +157,5 @@
         <ros2_control name="${name}" type="system">
             <hardware>
-                <plugin>gazebo_ros2_control/GazeboSystem</plugin>
+                <plugin>gz_ros2_control/GazeboSimSystem</plugin>
             </hardware>
             <joint name="${name}_hip_joint">

File: robots/descriptions/go2_description/xacro/velodyne.xacro (robot description, xacro)
@@ -47,11 +47,17 @@
         </visual>
     </link>
-    <!-- Gazebo requires the velodyne_gazebo_plugins package -->
+    <!-- Gazebo Harmonic has no velodyne_gazebo_plugins / libgazebo_ros_velodyne_laser.so.
+         The gpu_lidar sensor type produces the point cloud natively over gz
+         transport; champ_gazebo's ros_gz_bridge config
+         (config/velodyne_bridge.yaml) republishes it as a ROS 2
+         sensor_msgs/PointCloud2 on "velodyne_points". -->
     <gazebo reference="velodyne">
-        <sensor name="velodyne-VLP16" type="ray">
+        <sensor name="velodyne-VLP16" type="gpu_lidar">
         <pose>0 0 0 0 0 0</pose>
         <visualize>false</visualize>
         <update_rate>10</update_rate>
-        <ray>
+        <topic>velodyne_points</topic>
+        <gz_frame_id>velodyne</gz_frame_id>
+        <lidar>
             <scan>
             <horizontal>
@@ -69,6 +75,6 @@
             </scan>
             <range>
-            <min>0.3</min>
-            <max>131.0</max>
+            <min>0.9</min>
+            <max>130.0</max>
             <resolution>0.001</resolution>
             </range>
@@ -76,18 +82,7 @@
             <type>gaussian</type>
             <mean>0.0</mean>
-            <stddev>0.0</stddev>
+            <stddev>0.008</stddev>
             </noise>
-        </ray>
-        <plugin filename="libgazebo_ros_velodyne_laser.so" name="gazebo_ros_laser_controller">
-            <ros>
-              <namespace>/</namespace>
-              <remapping>~/out:=velodyne_points</remapping>
-            </ros>
-            <frame_name>velodyne</frame_name>
-            <organize_cloud>false</organize_cloud>
-            <min_range>0.9</min_range>
-            <max_range>130.0</max_range>
-            <gaussian_noise>0.008</gaussian_noise>
-        </plugin>
+        </lidar>
         </sensor>
     </gazebo>
