Commit message: Stand still on launch, disable contact sensors, stabilize Go2 sim
Make the quadruped hold a static stand until cmd_vel arrives (timeout +
deadband), publish gait-phase foot contacts instead of Gazebo contact
sensors, and fix effort-controller thrashing via retuned PID, stand-pose
initial joints, higher joint damping, and a softer trajectory horizon.

File: robots/descriptions/go2_description/xacro/const.xacro (robot description, xacro)
@@ -38,7 +38,11 @@
     <xacro:property name="calf_offset_y" value="0.0"/>
     <xacro:property name="calf_offset_z" value="-0.213"/>
-    <!-- joint limits -->
-    <xacro:property name="damping" value="0.01"/>
-    <xacro:property name="friction" value="0.2"/>
+    <!-- joint limits / passive dynamics (higher damping damps effort-PID thrashing) -->
+    <xacro:property name="damping" value="1.0"/>
+    <xacro:property name="friction" value="0.5"/>
+    <!-- Default stand pose matching champ quadruped_controller IK at nominal_height -->
+    <xacro:property name="stand_hip" value="0.0"/>
+    <xacro:property name="stand_thigh" value="1.0144"/>
+    <xacro:property name="stand_calf" value="-2.0287"/>
     <xacro:property name="hip_position_max" value="1.0472"/>
     <xacro:property name="hip_position_min" value="-1.0472"/>

File: robots/descriptions/go2_description/xacro/gazebo.xacro (robot description, xacro)
@@ -74,44 +74,8 @@
         </sensor>
     </gazebo>
-    <!-- Foot contact sensors, read by champ_gazebo's contact_sensor node via
-         ros_gz_bridge (see champ_gazebo/config/contact_bridge.yaml). Gazebo
-         Classic's contact state was read out-of-band via gazebo::transport;
-         Harmonic exposes it as a first-class <sensor type="contact">. -->
-    <gazebo reference="lf_foot_link">
-        <sensor name="lf_foot_contact" type="contact">
-            <always_on>true</always_on>
-            <update_rate>50</update_rate>
-            <contact>
-                <collision>lf_foot_link_collision</collision>
-            </contact>
-        </sensor>
-    </gazebo>
-    <gazebo reference="rf_foot_link">
-        <sensor name="rf_foot_contact" type="contact">
-            <always_on>true</always_on>
-            <update_rate>50</update_rate>
-            <contact>
-                <collision>rf_foot_link_collision</collision>
-            </contact>
-        </sensor>
-    </gazebo>
-    <gazebo reference="lh_foot_link">
-        <sensor name="lh_foot_contact" type="contact">
-            <always_on>true</always_on>
-            <update_rate>50</update_rate>
-            <contact>
-                <collision>lh_foot_link_collision</collision>
-            </contact>
-        </sensor>
-    </gazebo>
-    <gazebo reference="rh_foot_link">
-        <sensor name="rh_foot_contact" type="contact">
-            <always_on>true</always_on>
-            <update_rate>50</update_rate>
-            <contact>
-                <collision>rh_foot_link_collision</collision>
-            </contact>
-        </sensor>
-    </gazebo>
+    <!-- Foot contact sensors DISABLED. State estimation uses gait-phase
+         contacts published by quadruped_controller instead. Re-enable the
+         <sensor type="contact"> blocks and champ_gazebo contact_sensor /
+         contact_bridge if real sim contact feedback is needed. -->
     <!-- <gazebo reference="base_link">
         <turnGravityOff>false</turnGravityOff>

File: robots/descriptions/go2_description/xacro/leg.xacro (robot description, xacro)
@@ -160,17 +160,35 @@
             </hardware>
             <joint name="${name}_hip_joint">
-                <command_interface name="effort"/>
-                <state_interface name="position"/>
+                <command_interface name="effort">
+                    <param name="min">${-hip_torque_max}</param>
+                    <param name="max">${hip_torque_max}</param>
+                </command_interface>
+                <state_interface name="position">
+                    <param name="initial_value">${stand_hip}</param>
+                </state_interface>
                 <state_interface name="velocity"/>
+                <state_interface name="effort"/>
             </joint>
             <joint name="${name}_upper_leg_joint">
-                <command_interface name="effort"/>
-                <state_interface name="position"/>
+                <command_interface name="effort">
+                    <param name="min">${-thigh_torque_max}</param>
+                    <param name="max">${thigh_torque_max}</param>
+                </command_interface>
+                <state_interface name="position">
+                    <param name="initial_value">${stand_thigh}</param>
+                </state_interface>
                 <state_interface name="velocity"/>
+                <state_interface name="effort"/>
             </joint>
             <joint name="${name}_lower_leg_joint">
-                <command_interface name="effort"/>
-                <state_interface name="position"/>
+                <command_interface name="effort">
+                    <param name="min">${-calf_torque_max}</param>
+                    <param name="max">${calf_torque_max}</param>
+                </command_interface>
+                <state_interface name="position">
+                    <param name="initial_value">${stand_calf}</param>
+                </state_interface>
                 <state_interface name="velocity"/>
+                <state_interface name="effort"/>
             </joint>
         </ros2_control>
